Commit message: Fixed urdf

File: src/fanuc_description/robot/fanuc.urdf (robot description, URDF)
Before this commit: robot fanuc, 9 links, 8 joints
Links:
- removed link base_link
- added link link_0; collision mesh filename=package://fanuc_description/meshes/collision/link_0.stl; visual mesh filename=package://fanuc_description/meshes/visual/link_0.dae
Joints:
- joint joint_1: parent base_link -> link_0
- joint joint_5: origin xyz=0 0 0.835 rpy=1.5708 0 0 -> xyz=0 0 0.860 rpy=1.5708 0 0
- joint virtual_joint: child base_link -> link_0

Commit message: Added pkg

File: src/fanuc_description/robot/fanuc.urdf (robot description, URDF)
Before this commit: robot fanuc, 9 links, 8 joints
Links:
- removed link link_0
- added link base_link; collision mesh filename=package://fanuc_description/meshes/collision/link_0.stl; visual mesh filename=package://fanuc_description/meshes/visual/link_0.dae
Joints:
- joint joint_1: parent link_0 -> base_link
- joint virtual_joint: child link_0 -> base_link
